File: pixel_interface_v3/pixel_interface_v3.kicad_pcb (KiCad board)
At the start: 2 copper layers, 33.6 x 53.3 mm, 9 parts, among them J1 Analog, J2 POWER, J3 Digital/PWM, J4 D10_D9_D8, J5 YYZ_PIXEL

Commit message: final version of the pixel_interface board
Routing:
- added copper zone on B.Cu, net GND
- added copper zone on F.Cu, net GND
Other:
- outline, holes or cut-outs redrawn
