File: Hardware/yahrzeit_power_dist/yahrzeit_power_dist.kicad_pcb (KiCad board)
At the start: 2 copper layers, 300 x 100 mm, 27 parts, among them J1 12V Power In, J3 5V Power Out 1, J4 5V Power Out 2, J5 5V Power Out 3, J6 5V Power Out 4, J7 5V Power Out 5, J8 5V Power Out 6, U1 PTH12060WAH

Commit message: completed the power distribuiion board design
Parts:
- removed D1: REVERSE-POLARITY, Package_TO_SOT_THT:TO-220-2_Vertical
- removed D2: 15V TVS, Diode_SMD:D_SMB
- removed U1: PTH12060WAH, yahrzeit_power_dist:TI_PTH12060WAH_EUW_THT
- added LED1: POWER ON, LED_SMD:LED_0805_2012Metric, F.Cu at (121.0, 39.3)
- added TP2: GND, TestPoint:TestPoint_Pad_D2.5mm, F.Cu at (7.50, 33.0)
- added TP3: OUTPUT 5V, TestPoint:TestPoint_Pad_D2.5mm, F.Cu at (132.5, 17.0)
- C1: footprint Capacitor_SMD:CP_Elec_8x10.5 -> Capacitor_THT:CP_Radial_D10.0mm_P5.00mm
- C2: value 1000uF 10V SMD -> 22uF; footprint Capacitor_SMD:CP_Elec_10x10.5 -> Capacitor_SMD:C_1210_3225Metric
- C3: value 470uF -> 0.1uF; footprint Capacitor_SMD:CP_Elec_8x10.5 -> Capacitor_SMD:C_0805_2012Metric
- F1: value 4A SLOW -> 7.5A MINI BLADE
- F2, F3, F4, F5, F6, F7: value 1.25A SLOW -> 1.5A HOLD PTC
- J1: value 12V Power In -> 5V Power In; footprint Connector_JST:JST_VH_B3P-VH-B_1x03_P3.96mm_Vertical -> Connector_JST:JST_VH_B3P-VH_1x03_P3.96mm_Vertical
- R1: value 280R 1% -> 1K
- TP1: value +5V Test -> +5V; footprint yahrzeit_power_dist:TestPoint_Keystone_5016_Compact -> TestPoint:TestPoint_Pad_D2.5mm
- TP4: renamed from TP2; value GND Test -> OUTPUT GND; footprint yahrzeit_power_dist:TestPoint_Keystone_5016_Compact -> TestPoint:TestPoint_Pad_D2.5mm
- moved TP1 269.6 mm to (7.50, 17.0)
- moved H4 167.6 mm to (132.5, 42.5)
- moved H2 160.0 mm to (132.5, 7.50)
- moved F7 157.0 mm to (118.0, 20.0), turned to -90 degrees
- moved J7 155.0 mm to (118.0, 8.00)
- moved TP4 145.1 mm to (132.5, 33.0)
- moved F6 127.0 mm to (98.0, 20.0), turned to -90 degrees
- moved J6 125.0 mm to (98.0, 8.00)
- moved F5 97.0 mm to (78.0, 20.0), turned to -90 degrees
- moved J5 95.0 mm to (78.0, 8.00)
- moved C2 71.3 mm to (107.0, 34.5), turned to -90 degrees
- moved F4 67.1 mm to (58.0, 20.0), turned to -90 degrees
- moved J4 65.0 mm to (58.0, 8.00)
- moved C1 63.0 mm to (96.6, 32.0), turned to -90 degrees
- moved F1 60.3 mm to (81.7, 30.0), turned to -90 degrees
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- renumbered J3 to J2, J4 to J3, J5 to J4, J6 to J5, J7 to J6, J8 to J7
Connections:
- C1 pad 1: /+12V_RECTIFIED -> /+5V_BUS
- C3 pad 1: /+12V_RECTIFIED -> /+5V_BUS
- F1 pad 1: Net-(D1-A) -> /+5V_BUS
- R1 pad 1: Net-(U1-ADJ) -> /+5V_BUS
- R1 pad 2: GND -> Net-(LED1-A)
- TP1 pad 1: /+5V_BUS -> Net-(J1-Pin_1)
Routing:
- net Net-(J1-Pin_1): track 0.00 -> 97.5 mm
- net Net-(J7-Pin_1): track 0.00 -> 24.7 mm
- net Net-(J6-Pin_1): track 0.00 -> 9.86 mm
- net Net-(J5-Pin_1): track 0.00 -> 9.86 mm
- net Net-(J4-Pin_1): track 0.00 -> 9.86 mm
- net Net-(J3-Pin_1): track 0.00 -> 9.86 mm
- net Net-(J2-Pin_1): track 0.00 -> 9.86 mm
- net /+5V_BUS: track 0.00 -> 3.40 mm
- net Net-(LED1-A): track 0.00 -> 2.65 mm
- added copper zone on F.Cu, net /+5V_BUS
- added copper zone on B.Cu, net GND
- added copper zone on F.Cu, net GND
Other:
- board size 300 x 100 mm -> 140 x 50 mm
- board text added: "1.5A PTC"
- board text added: "5V POWER INPUT"
- board text added: "INPUT +5V"
- board text added: "INPUT FUSE - 7.5A"
- board text added: "INPUT GND"
- board text added: "OUT 6 +5V"
- board text added: "OUTPUT GND"
- board text added: "POWERED"
- board text removed: "+12V"
- board text removed: "+5V TEST"
- board text removed: "1.25A PTC"
- board text removed: "12V FILTER"
- board text removed: "12V POWER INPUT"
- board text removed: "12V TVS"
- board text removed: "12V+"
- board text removed: "5V BUCK - PTH12060WAH"
- board text removed: "5V FILTER"
- board text removed: "5V+"
- board text removed: "GND TEST"
- board text removed: "INPUT FUSE - 4A"
- board text removed: "REVERSE-POLARITY DIODE"

Commit message: new approach to cables
Parts:
- J1: value 5V Power In -> Power IN; footprint Connector_JST:JST_VH_B3P-VH_1x03_P3.96mm_Vertical -> yahrzeit_power_dist:TerminalBlock_Phoenix_BC-508X10-2_1x02_P5.08mm_Horizontal
- J2: value 5V Power Out 1 -> Power Out; footprint Connector_JST:JST_VH_B2P-VH-B_1x02_P3.96mm_Vertical -> yahrzeit_power_dist:TerminalBlock_Phoenix_BC-508X10-2_1x02_P5.08mm_Horizontal
- J3: value 5V Power Out 2 -> Power Out; footprint Connector_JST:JST_VH_B2P-VH-B_1x02_P3.96mm_Vertical -> yahrzeit_power_dist:TerminalBlock_Phoenix_BC-508X10-2_1x02_P5.08mm_Horizontal
- J4: value 5V Power Out 3 -> Power Out; footprint Connector_JST:JST_VH_B2P-VH-B_1x02_P3.96mm_Vertical -> yahrzeit_power_dist:TerminalBlock_Phoenix_BC-508X10-2_1x02_P5.08mm_Horizontal
- J5: value 5V Power Out 4 -> Power Out; footprint Connector_JST:JST_VH_B2P-VH-B_1x02_P3.96mm_Vertical -> yahrzeit_power_dist:TerminalBlock_Phoenix_BC-508X10-2_1x02_P5.08mm_Horizontal
- J6: value 5V Power Out 5 -> Power Out; footprint Connector_JST:JST_VH_B2P-VH-B_1x02_P3.96mm_Vertical -> yahrzeit_power_dist:TerminalBlock_Phoenix_BC-508X10-2_1x02_P5.08mm_Horizontal
- J7: value 5V Power Out 6 -> Power Out; footprint Connector_JST:JST_VH_B2P-VH-B_1x02_P3.96mm_Vertical -> yahrzeit_power_dist:TerminalBlock_Phoenix_BC-508X10-2_1x02_P5.08mm_Horizontal
- TP3: value OUTPUT 5V -> OUT6 5V
- moved J2 5.10 mm to (23.0, 9.00), turned to 180 degrees
- moved J3 5.10 mm to (43.0, 9.00), turned to 180 degrees
- moved J4 5.10 mm to (63.0, 9.00), turned to 180 degrees
- moved J5 5.10 mm to (83.0, 9.00), turned to 180 degrees
- moved J6 5.10 mm to (103.0, 9.00), turned to 180 degrees
- moved J7 5.10 mm to (123.0, 9.00), turned to 180 degrees
- moved F2 5.00 mm to (23.0, 20.0)
- moved F3 5.00 mm to (43.0, 20.0)
- moved F4 5.00 mm to (63.0, 20.0)
- moved F5 5.00 mm to (83.0, 20.0)
- moved F6 5.00 mm to (103.0, 20.0)
- moved F7 5.00 mm to (123.0, 20.0)
- moved J1 0.10 mm to (55.9, 38.0)
Connections:
- J1 pad 2: unconnected-(J1-Pin_2-Pad2) -> GND
Routing:
- net Net-(J7-Pin_1): track 24.7 -> 18.7 mm
- net Net-(J6-Pin_1): track 9.86 -> 8.86 mm
- net Net-(J5-Pin_1): track 9.86 -> 8.86 mm
- net Net-(J4-Pin_1): track 9.86 -> 8.86 mm
- net Net-(J3-Pin_1): track 9.86 -> 8.86 mm
- net Net-(J2-Pin_1): track 9.86 -> 8.86 mm
Other:
- board text added: "A"
- board text added: "POWER INPUT"
- board text added: "YAHRZEIT WALL POWER DISTRIBUTION REV A - OCTOBER 2026 ALLAN M SCHWARTZ"
- board text removed: "5V POWER INPUT"
- board text removed: "INPUT GND"
- board text removed: "NC"
- board text removed: "OUTPUT GND"
- board text removed: "YAHRZEIT WALL POWER DISTRIBUTION REV A - SEPTEMBER 2026 ALLAN M SCHWARTZ"
