File: Hardware/yahrzeit_power_dist/yahrzeit_power_dist.kicad_sch (KiCad schematic)
At the start: 23 parts, among them J1 12V Power In, J3 5V Power Out 1, J4 5V Power Out 2, J5 5V Power Out 3, J6 5V Power Out 4, J7 5V Power Out 5, J8 5V Power Out 6, U1 PTH12060WAH

Commit message: completed the power distribuiion board design
Parts:
- removed D1: REVERSE-POLARITY, Package_TO_SOT_THT:TO-220-2_Vertical, symbol Device:D_Schottky
- removed D2: 15V TVS, Diode_SMD:D_SMB, symbol Device:D_TVS
- removed U1: PTH12060WAH, yahrzeit_power_dist:TI_PTH12060WAH_EUW_THT, symbol yahrzeit_power_dist:PTH12060WAH
- added LED1: POWER ON, LED_SMD:LED_0805_2012Metric, symbol Device:LED
- added TP2: GND, TestPoint:TestPoint_Pad_D2.5mm, symbol Connector:TestPoint
- added TP3: OUT6 5V, TestPoint:TestPoint_Pad_D2.5mm, symbol Connector:TestPoint
- C1: footprint Capacitor_SMD:CP_Elec_8x10.5 -> Capacitor_THT:CP_Radial_D10.0mm_P5.00mm; MPN EEE-FT1E471AV -> 25ZLH470MEFC10X12.5
- C2: renamed from C3; value 470uF -> 22uF; footprint Capacitor_SMD:CP_Elec_8x10.5 -> Capacitor_SMD:C_1210_3225Metric; symbol Device:C_Polarized -> Device:C_Small; MPN EEE-FT1E471AV -> GMC32X7R226K25NT
- C3: renamed from C2; value 1000uF 10V SMD -> 0.1uF 50V X7R; footprint Capacitor_SMD:CP_Elec_10x10.5 -> Capacitor_SMD:C_0805_2012Metric; symbol Device:C_Polarized -> Device:C_Small; MPN EEE-FP1A102AP -> CC0805KRX7R9BB104
- F1: value 4A SLOW -> 7.5A MINI BLADE; MPN 0215004.MXP -> 0297007.WXNV
- F2, F3, F4, F5, F6, F7: value 1.25A SLOW -> 1.5A HOLD PTC
- J1: value 12V Power In -> 5V Power In; footprint Connector_JST:JST_VH_B3P-VH-B_1x03_P3.96mm_Vertical -> Connector_JST:JST_VH_B3P-VH_1x03_P3.96mm_Vertical; MPN JST B3P-VH -> B3P-VH
- R1: value 280R 1% -> 1K; MPN RC0805FR-07280RL -> RC0805FR-071KL
- TP1: value +5V Test -> +5V; footprint yahrzeit_power_dist:TestPoint_Keystone_5016_Compact -> TestPoint:TestPoint_Pad_D2.5mm; MPN Keystone 5016 -> PCB test pad
- TP4: renamed from TP2; value GND Test -> OUTPUT GND; footprint yahrzeit_power_dist:TestPoint_Keystone_5016_Compact -> TestPoint:TestPoint_Pad_D2.5mm; MPN Keystone 5016 -> PCB test pad
- renumbered J3 to J2, J4 to J3, J5 to J4, J6 to J5, J7 to J6, J8 to J7
Connections:
- net +12V_RECTIFIED is gone; now on net +5V_BUS: C1.1, C2.1
- net +5V_BUS: now also F1.1, R1.1; no longer TP1.1
- net GND: now also LED1.1 (K), TP2.1; no longer R1.2
- net at F1.2, J1.1 (Pin_1): now also TP1.1
- net at F7.1, J7.1 (Pin_1): now also TP3.1
- new net: LED1.2 (A), R1.2
- no-connect marks 5 -> 1
Other:
- note added: "5 V INPUT / PROTECTION"
- note added: "DESIGN NOTES: 1. Board distributes regulated 5 V power for one panel column (six branches of 56 LEDs). 2. F1 is a 7.5 A replaceable input fuse; F2-F7 are 1.5 A hold resettable branch protectors. 3. C1/C2/C3 provide complementary bulk, mid-frequency, and high-frequency bypassing. 4. Each YYZ_PIXEL chain also provides local bulk and IC decoupling at its load. 5. Use 2 oz copper, broad +5V/GND pours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"
- note added: "bulk, mid-freq., high-freq. bypass"
- note removed: "12 V INPUT / PROTECTION"
- note removed: "DESIGN NOTES: 1. Board distributes power for one panel column (six branches of 56 LEDs). 2. U1 is TI PTH12060WAH, configured for regulated 5.0 V output. 3. F1 and F2-F7 are starting values only; confirm from measured operating/inrush current. 4. Use 2 oz copper, broad +5V/GND pours, short high-current paths, and 2.0 mm FR-4. 5. D1 must be selected/rated for full input current; an ideal-diode MOSF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"
- note removed: "TI PTH12060WAH BUCK MODULE (10 A)"
- note removed: "U1: TI PTH12060WAH through-hole buck module. R1 = 280 ohm sets 5.0 V. Leave INHIBIT, TRACK, MARGIN UP and MARGIN DOWN open for normal operation."
- moved on the sheet: C1, F1, F2, F3, F4, F5, F6, F7, J1, J2, J3, J4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

Commit message: new approach to cables
Parts:
- removed J1: 5V Power In, Connector_JST:JST_VH_B3P-VH_1x03_P3.96mm_Vertical, symbol Connector_Generic:Conn_01x03
- added J1: Power IN, yahrzeit_power_dist:TerminalBlock_Phoenix_BC-508X10-2_1x02_P5.08mm_Horizontal, symbol Connector_Generic:Conn_01x02
- F1: MPN 0297007.WXNV -> 029707.5WXNV
- J2: value 5V Power Out 1 -> Power Out; footprint Connector_JST:JST_VH_B2P-VH-B_1x02_P3.96mm_Vertical -> yahrzeit_power_dist:TerminalBlock_Phoenix_BC-508X10-2_1x02_P5.08mm_Horizontal; MPN JST B2P-VH -> Phoenix Contact 5442206
- J3: value 5V Power Out 2 -> Power Out; footprint Connector_JST:JST_VH_B2P-VH-B_1x02_P3.96mm_Vertical -> yahrzeit_power_dist:TerminalBlock_Phoenix_BC-508X10-2_1x02_P5.08mm_Horizontal; MPN JST B2P-VH -> Phoenix Contact 5442206
- J4: value 5V Power Out 3 -> Power Out; footprint Connector_JST:JST_VH_B2P-VH-B_1x02_P3.96mm_Vertical -> yahrzeit_power_dist:TerminalBlock_Phoenix_BC-508X10-2_1x02_P5.08mm_Horizontal; MPN JST B2P-VH -> Phoenix Contact 5442206
- J5: value 5V Power Out 4 -> Power Out; footprint Connector_JST:JST_VH_B2P-VH-B_1x02_P3.96mm_Vertical -> yahrzeit_power_dist:TerminalBlock_Phoenix_BC-508X10-2_1x02_P5.08mm_Horizontal; MPN JST B2P-VH -> Phoenix Contact 5442206
- J6: value 5V Power Out 5 -> Power Out; footprint Connector_JST:JST_VH_B2P-VH-B_1x02_P3.96mm_Vertical -> yahrzeit_power_dist:TerminalBlock_Phoenix_BC-508X10-2_1x02_P5.08mm_Horizontal; MPN JST B2P-VH -> Phoenix Contact 5442206
- J7: value 5V Power Out 6 -> Power Out; footprint Connector_JST:JST_VH_B2P-VH-B_1x02_P3.96mm_Vertical -> yahrzeit_power_dist:TerminalBlock_Phoenix_BC-508X10-2_1x02_P5.08mm_Horizontal; MPN JST B2P-VH -> Phoenix Contact 5442206
Connections:
- net GND: now also J1.2 (Pin_2)
- net at F1.2, TP1.1: now also J1.1 (Pin_1)
- no-connect marks 1 -> 0
